Commit message: added args to use abs paths for root and meshes

File: dagana_urdf/urdf/dagana.urdf.xacro (robot description, xacro)
@@ -1,5 +1,7 @@
 <?xml version="1.0"?>
 <robot xmlns:xacro="http://ros.org/wiki/xacro" name="dagana">
-<xacro:include filename="$(find dagana_urdf)/urdf/dagana_macro.urdf.xacro" />
+<xacro:arg name="dagana_root" default="$(find dagana_urdf)" />
+<xacro:property name="DAGANA_ROOT" value="$(arg dagana_root)" />
+<xacro:include filename="${DAGANA_ROOT}/urdf/dagana_macro.urdf.xacro" />
 <link name="world"/>
 <joint name="virtualFixed" type="fixed">

File: dagana_urdf/urdf/dagana_macro.urdf.xacro (robot description, xacro)
@@ -1,5 +1,25 @@
 <?xml version="1.0"?>
 <robot xmlns:xacro="http://ros.org/wiki/xacro">
-<xacro:include filename="$(find dagana_urdf)/urdf/config/dagana_config.urdf.xacro" />
+<xacro:arg name="dagana_root" default="$(find dagana_urdf)" />
+<xacro:property name="DAGANA_ROOT" value="$(arg dagana_root)" />
+<!-- setting use_abs_mesh_paths should be kept to false
+for use with tools like RViz, which does not accept plain
+abolute paths for mesh paths-->
+<xacro:arg name="use_abs_mesh_paths" default="false" />
+<xacro:arg name="use_local_filesys_for_meshes" default="false" />
+<xacro:property name="USE_ABS_MESH_PATHS" value="$(arg use_abs_mesh_paths)" />
+<xacro:property name="USE_LOCAL_FILESYS_FOR_MESHES" value="$(arg use_local_filesys_for_meshes)" />
+<xacro:if value="${USE_ABS_MESH_PATHS}">
+    <xacro:if value="${USE_LOCAL_FILESYS_FOR_MESHES}">
+    <xacro:property name="DAGANA_MESH_PATH" value="file://${DAGANA_ROOT}/meshes" />
+    </xacro:if>
+    <xacro:unless value="${USE_LOCAL_FILESYS_FOR_MESHES}">
+    <xacro:property name="DAGANA_MESH_PATH" value="${DAGANA_ROOT}/meshes" />
+    </xacro:unless>
+</xacro:if>
+<xacro:unless value="${USE_ABS_MESH_PATHS}">
+    <xacro:property name="DAGANA_MESH_PATH" value="package://dagana_urdf/meshes" />
+</xacro:unless>
+<xacro:include filename="${DAGANA_ROOT}/urdf/config/dagana_config.urdf.xacro" />
 <xacro:macro name="dagana_gripper" params="name joint_type parent_link GAZEBO_URDF:=^|false *origin">
     <joint name="${name}_mount_joint" type="fixed">
@@ -23,12 +43,12 @@
                 <origin xyz="0 0 0" rpy="0 0 0" />
                 <geometry>
-                    <mesh filename="package://dagana_urdf/meshes/dg0001-simplified.stl" scale="${mmTom} ${mmTom} ${mmTom}" />
-                </geometry>
-                <material name="dagana_dark_grey"/>
-            </visual>
-            <collision>
-                <origin xyz="0 0 0" rpy="0 0 0" />
-                <geometry>
-                    <mesh filename="package://dagana_urdf/meshes/dg0001-simplified_v2.stl" scale="${mmTom} ${mmTom} ${mmTom}" />
+                    <mesh filename="${DAGANA_MESH_PATH}/dg0001-simplified.stl" scale="${mmTom} ${mmTom} ${mmTom}" />
+                </geometry>
+                <material name="dagana_dark_grey"/>
+            </visual>
+            <collision>
+                <origin xyz="0 0 0" rpy="0 0 0" />
+                <geometry>
+                    <mesh filename="${DAGANA_MESH_PATH}/dg0001-simplified_v2.stl" scale="${mmTom} ${mmTom} ${mmTom}" />
                 </geometry>
             </collision>
@@ -49,12 +69,12 @@
                 <origin xyz="0 0 0" rpy="0 0 0" />
                 <geometry>
-                    <mesh filename="package://dagana_urdf/meshes/dagana_fixed_A.stl" scale="${mmTom} ${mmTom} ${mmTom}" />
-                </geometry>
-                <material name="dagana_dark_grey"/>
-            </visual>
-            <collision>
-                <origin xyz="0 0 0" rpy="0 0 0" />
-                <geometry>
-                    <mesh filename="package://dagana_urdf/meshes/dagana_fixed_A_simple.stl" scale="${mmTom} ${mmTom} ${mmTom}" />
+                    <mesh filename="${DAGANA_MESH_PATH}/dagana_fixed_A.stl" scale="${mmTom} ${mmTom} ${mmTom}" />
+                </geometry>
+                <material name="dagana_dark_grey"/>
+            </visual>
+            <collision>
+                <origin xyz="0 0 0" rpy="0 0 0" />
+                <geometry>
+                    <mesh filename="${DAGANA_MESH_PATH}/dagana_fixed_A_simple.stl" scale="${mmTom} ${mmTom} ${mmTom}" />
                 </geometry>
             </collision>
@@ -74,12 +94,12 @@
                 <origin xyz="0 0 0" rpy="0 0 0" />
                 <geometry>
-                    <mesh filename="package://dagana_urdf/meshes/mesh_dagana-base_simple.stl" scale="${mmTom} ${mmTom} ${mmTom}" />
-                </geometry>
-                <material name="dagana_dark_grey"/>
-            </visual>
-            <collision>
-                <origin xyz="0 0 0" rpy="0 0 0" />
-                <geometry>
-                    <mesh filename="package://dagana_urdf/meshes/mesh_dagana-base_ch.stl" scale="${mmTom} ${mmTom} ${mmTom}" />
+                    <mesh filename="${DAGANA_MESH_PATH}/mesh_dagana-base_simple.stl" scale="${mmTom} ${mmTom} ${mmTom}" />
+                </geometry>
+                <material name="dagana_dark_grey"/>
+            </visual>
+            <collision>
+                <origin xyz="0 0 0" rpy="0 0 0" />
+                <geometry>
+                    <mesh filename="${DAGANA_MESH_PATH}/mesh_dagana-base_ch.stl" scale="${mmTom} ${mmTom} ${mmTom}" />
                 </geometry>
             </collision>
@@ -96,12 +116,12 @@
                 <origin xyz="0 0 0" rpy="0 0 0" />
                 <geometry>
-                    <mesh filename="package://dagana_urdf/meshes/dagana_fixed_B.stl" scale="${mmTom} ${mmTom} ${mmTom}" />
-                </geometry>
-                <material name="dagana_dark_grey"/>
-            </visual>
-            <collision>
-                <origin xyz="0 0 0" rpy="0 0 0" />
-                <geometry>
-                    <mesh filename="package://dagana_urdf/meshes/dagana_fixed_B_simple.stl" scale="${mmTom} ${mmTom} ${mmTom}" />
+                    <mesh filename="${DAGANA_MESH_PATH}/dagana_fixed_B.stl" scale="${mmTom} ${mmTom} ${mmTom}" />
+                </geometry>
+                <material name="dagana_dark_grey"/>
+            </visual>
+            <collision>
+                <origin xyz="0 0 0" rpy="0 0 0" />
+                <geometry>
+                    <mesh filename="${DAGANA_MESH_PATH}/dagana_fixed_B_simple.stl" scale="${mmTom} ${mmTom} ${mmTom}" />
                 </geometry>
             </collision>
@@ -116,12 +136,12 @@
                 <origin xyz="0 0 0" rpy="0 0 0" />
                 <geometry>
-                    <mesh filename="package://dagana_urdf/meshes/dagana_fixed_C.stl" scale="${mmTom} ${mmTom} ${mmTom}" />
-                </geometry>
-                <material name="dagana_dark_grey"/>
-            </visual>
-            <collision>
-                <origin xyz="0 0 0" rpy="0 0 0" />
-                <geometry>
-                    <mesh filename="package://dagana_urdf/meshes/dagana_fixed_C_simple.stl" scale="${mmTom} ${mmTom} ${mmTom}" />
+                    <mesh filename="${DAGANA_MESH_PATH}/dagana_fixed_C.stl" scale="${mmTom} ${mmTom} ${mmTom}" />
+                </geometry>
+                <material name="dagana_dark_grey"/>
+            </visual>
+            <collision>
+                <origin xyz="0 0 0" rpy="0 0 0" />
+                <geometry>
+                    <mesh filename="${DAGANA_MESH_PATH}/dagana_fixed_C_simple.stl" scale="${mmTom} ${mmTom} ${mmTom}" />
                 </geometry>
             </collision>
@@ -161,12 +181,12 @@
                 <origin xyz="0 0 0" rpy="0 0 0" />
                 <geometry>
-                    <mesh filename="package://dagana_urdf/meshes/dg0002.stl" scale="${mmTom} ${mmTom} ${mmTom}" />
-                </geometry>
-                <material name="dagana_dark_grey"/>
-            </visual>
-            <collision>
-                <origin xyz="0 0 0" rpy="0 0 0" />
-                <geometry>
-                    <mesh filename="package://dagana_urdf/meshes/dg0002-ch.stl" scale="${mmTom} ${mmTom} ${mmTom}" />
+                    <mesh filename="${DAGANA_MESH_PATH}/dg0002.stl" scale="${mmTom} ${mmTom} ${mmTom}" />
+                </geometry>
+                <material name="dagana_dark_grey"/>
+            </visual>
+            <collision>
+                <origin xyz="0 0 0" rpy="0 0 0" />
+                <geometry>
+                    <mesh filename="${DAGANA_MESH_PATH}/dg0002-ch.stl" scale="${mmTom} ${mmTom} ${mmTom}" />
                 </geometry>
             </collision>
@@ -186,12 +206,12 @@
                 <origin xyz="0 0 0" rpy="0 0 0" />
                 <geometry>
-                    <mesh filename="package://dagana_urdf/meshes/dagana_claw_A.stl" scale="${mmTom} ${mmTom} ${mmTom}" />
-                </geometry>
-                <material name="dagana_dark_grey"/>
-            </visual>
-            <collision>
-                <origin xyz="0 0 0" rpy="0 0 0" />
-                <geometry>
-                    <mesh filename="package://dagana_urdf/meshes/dagana_claw_A_simple.stl" scale="${mmTom} ${mmTom} ${mmTom}" />
+                    <mesh filename="${DAGANA_MESH_PATH}/dagana_claw_A.stl" scale="${mmTom} ${mmTom} ${mmTom}" />
+                </geometry>
+                <material name="dagana_dark_grey"/>
+            </visual>
+            <collision>
+                <origin xyz="0 0 0" rpy="0 0 0" />
+                <geometry>
+                    <mesh filename="${DAGANA_MESH_PATH}/dagana_claw_A_simple.stl" scale="${mmTom} ${mmTom} ${mmTom}" />
                 </geometry>
             </collision>
@@ -211,12 +231,12 @@
                 <origin xyz="0 0 0" rpy="0 0 0" />
                 <geometry>
-                    <mesh filename="package://dagana_urdf/meshes/mesh_dagana-link_simple.stl" scale="${mmTom} ${mmTom} ${mmTom}" />
-                </geometry>
-                <material name="dagana_dark_grey"/>
-            </visual>
-            <collision>
-                <origin xyz="0 0 0" rpy="0 0 0" />
-                <geometry>
-                    <mesh filename="package://dagana_urdf/meshes/mesh_dagana-link_ch.stl" scale="${mmTom} ${mmTom} ${mmTom}" />
+                    <mesh filename="${DAGANA_MESH_PATH}/mesh_dagana-link_simple.stl" scale="${mmTom} ${mmTom} ${mmTom}" />
+                </geometry>
+                <material name="dagana_dark_grey"/>
+            </visual>
+            <collision>
+                <origin xyz="0 0 0" rpy="0 0 0" />
+                <geometry>
+                    <mesh filename="${DAGANA_MESH_PATH}/mesh_dagana-link_ch.stl" scale="${mmTom} ${mmTom} ${mmTom}" />
                 </geometry>
             </collision>
@@ -233,12 +253,12 @@
                 <origin xyz="0 0 0" rpy="0 0 0" />
                 <geometry>
-                    <mesh filename="package://dagana_urdf/meshes/dagana_claw_B.stl" scale="${mmTom} ${mmTom} ${mmTom}" />
-                </geometry>
-                <material name="dagana_dark_grey"/>
-            </visual>
-            <collision>
-                <origin xyz="0 0 0" rpy="0 0 0" />
-                <geometry>
-                    <mesh filename="package://dagana_urdf/meshes/dagana_claw_B_simple.stl" scale="${mmTom} ${mmTom} ${mmTom}" />
+                    <mesh filename="${DAGANA_MESH_PATH}/dagana_claw_B.stl" scale="${mmTom} ${mmTom} ${mmTom}" />
+                </geometry>
+                <material name="dagana_dark_grey"/>
+            </visual>
+            <collision>
+                <origin xyz="0 0 0" rpy="0 0 0" />
+                <geometry>
+                    <mesh filename="${DAGANA_MESH_PATH}/dagana_claw_B_simple.stl" scale="${mmTom} ${mmTom} ${mmTom}" />
                 </geometry>
             </collision>
@@ -295,12 +315,12 @@
                 <origin xyz="0 0 0" rpy="0 0 0" />
                 <geometry>
-                    <mesh filename="package://dagana_urdf/meshes/mesh_formwork-base.stl" scale="${mmTom} ${mmTom} ${mmTom}" />
-                </geometry>
-                <material name="dagana_dark_grey"/>
-            </visual>
-            <collision>
-                <origin xyz="0 0 0" rpy="0 0 0" />
-                <geometry>
-                    <mesh filename="package://dagana_urdf/meshes/mesh_formwork-base_ch.stl" scale="${mmTom} ${mmTom} ${mmTom}" />
+                    <mesh filename="${DAGANA_MESH_PATH}/mesh_formwork-base.stl" scale="${mmTom} ${mmTom} ${mmTom}" />
+                </geometry>
+                <material name="dagana_dark_grey"/>
+            </visual>
+            <collision>
+                <origin xyz="0 0 0" rpy="0 0 0" />
+                <geometry>
+                    <mesh filename="${DAGANA_MESH_PATH}/mesh_formwork-base_ch.stl" scale="${mmTom} ${mmTom} ${mmTom}" />
                 </geometry>
             </collision>
@@ -320,12 +340,12 @@
                 <origin xyz="0 0 0" rpy="0 0 0" />
                 <geometry>
-                    <mesh filename="package://dagana_urdf/meshes/mesh_formwork-thumb.stl" scale="${mmTom} ${mmTom} ${mmTom}" />
-                </geometry>
-                <material name="dagana_dark_grey"/>
-            </visual>
-            <collision>
-                <origin xyz="0 0 0" rpy="0 0 0" />
-                <geometry>
-                    <mesh filename="package://dagana_urdf/meshes/mesh_formwork-thumb_ch.stl" scale="${mmTom} ${mmTom} ${mmTom}" />
+                    <mesh filename="${DAGANA_MESH_PATH}/mesh_formwork-thumb.stl" scale="${mmTom} ${mmTom} ${mmTom}" />
+                </geometry>
+                <material name="dagana_dark_grey"/>
+            </visual>
+            <collision>
+                <origin xyz="0 0 0" rpy="0 0 0" />
+                <geometry>
+                    <mesh filename="${DAGANA_MESH_PATH}/mesh_formwork-thumb_ch.stl" scale="${mmTom} ${mmTom} ${mmTom}" />
                 </geometry>
             </collision>
@@ -347,12 +367,12 @@
                 <origin xyz="0 0 0" rpy="0 0 0" />
                 <geometry>
-                    <mesh filename="package://dagana_urdf/meshes/mesh_tube-thumb_simple.stl" scale="${mmTom} ${mmTom} ${mmTom}" />
-                </geometry>
-                <material name="dagana_dark_grey"/>
-            </visual>
-            <collision>
-                <origin xyz="0 0 0" rpy="0 0 0" />
-                <geometry>
-                    <mesh filename="package://dagana_urdf/meshes/mesh_tube-thumb_ch.stl" scale="${mmTom} ${mmTom} ${mmTom}" />
+                    <mesh filename="${DAGANA_MESH_PATH}/mesh_tube-thumb_simple.stl" scale="${mmTom} ${mmTom} ${mmTom}" />
+                </geometry>
+                <material name="dagana_dark_grey"/>
+            </visual>
+            <collision>
+                <origin xyz="0 0 0" rpy="0 0 0" />
+                <geometry>
+                    <mesh filename="${DAGANA_MESH_PATH}/mesh_tube-thumb_ch.stl" scale="${mmTom} ${mmTom} ${mmTom}" />
                 </geometry>
             </collision>
@@ -372,12 +392,12 @@
                 <origin xyz="0 0 0" rpy="0 0 0" />
                 <geometry>
-                    <mesh filename="package://dagana_urdf/meshes/mesh_tube-base_simple.stl" scale="${mmTom} ${mmTom} ${mmTom}" />
-                </geometry>
-                <material name="dagana_dark_grey"/>
-            </visual>
-            <collision>
-                <origin xyz="0 0 0" rpy="0 0 0" />
-                <geometry>
-                    <mesh filename="package://dagana_urdf/meshes/mesh_tube-base_ch.stl" scale="${mmTom} ${mmTom} ${mmTom}" />
+                    <mesh filename="${DAGANA_MESH_PATH}/mesh_tube-base_simple.stl" scale="${mmTom} ${mmTom} ${mmTom}" />
+                </geometry>
+                <material name="dagana_dark_grey"/>
+            </visual>
+            <collision>
+                <origin xyz="0 0 0" rpy="0 0 0" />
+                <geometry>
+                    <mesh filename="${DAGANA_MESH_PATH}/mesh_tube-base_ch.stl" scale="${mmTom} ${mmTom} ${mmTom}" />
                 </geometry>
             </collision>
